File: Thesis Work/Layout/PCB Design/Eagle/DM & CM/DMP.brd (EAGLE design)
At the start: 37.8 x 18.2 mm, 5 parts

Commit message: c
Parts:
- added J1, J2: SMA-J-P-H-ST-EM1, SMA:SAMTEC_SMA-J-P-H-ST-EM1
- moved C3 0.08 mm to (51.9, 24.9)
Connections:
- removed net N$6: C2.1, C4.1, CHIP.3
- removed net N$7: C1.1, CHIP.4
- new net GND: C1.1, C2.1, C4.1, CHIP.3, CHIP.4
- net N$3: now also J1.1
- net N$4: now also J2.1
Routing:
- net GND: track 0.00 -> 35.5 mm, vias 0 -> 7
- net N$6: track 16.5 -> 0.00 mm
- net N$7: track 13.3 -> 0.00 mm
- net N$4: track 16.5 -> 23.3 mm
- net N$3: track 13.1 -> 18.5 mm
- added copper zone on layer 16, net GND
Other:
- board outline removed
