File: Thesis Work/Layout/PCB Design/Eagle/DM & CM/DMP.sch (EAGLE design)
At the start: 5 parts

Commit message: c
Parts:
- added J1, J2: SMA-J-P-H-ST-EM1, SMA:SMA-J-P-H-ST-EM1
Connections:
- removed net N$6: C2.1, C4.1, CHIP.3
- removed net N$7: C1.1, CHIP.4
- new net GND: C1.1, C2.1, C4.1, CHIP.3, CHIP.4
- net N$3: now also J1.1
- net N$4: now also J2.1
Changed lines of the file:
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@@
 <part name="C3" library="capa" deviceset="CAPA" device="1206"/>
 <part name="C4" library="capa" deviceset="CAPA" device="1206"/>
+<part name="J1" library="SMA" deviceset="SMA-J-P-H-ST-EM1" device=""/>
+<part name="J2" library="SMA" deviceset="SMA-J-P-H-ST-EM1" device=""/>
+<part name="GND1" library="supply1" library_urn="urn:adsk.eagle:library:371" deviceset="GND" device=""/>
+<part name="GND2" library="supply1" library_urn="urn:adsk.eagle:library:371" deviceset="GND" device=""/>
 </parts>
 <sheets>
@@
 <attribute name="VALUE" x="-1697.66" y="-894.68" size="1.778" layer="96"/>
 </instance>
+<instance part="J1" gate="G$1" x="-1818.1" y="-865.8" smashed="yes">
+<attribute name="NAME" x="-1821.91" y="-861.736" size="1.778" layer="95"/>
+<attribute name="VALUE" x="-1822.164" y="-870.118" size="1.778" layer="96"/>
+</instance>
+<instance part="J2" gate="G$1" x="-1684.5" y="-860.6" smashed="yes" rot="R180">
+<attribute name="NAME" x="-1680.69" y="-864.664" size="1.778" layer="95" rot="R180"/>
+<attribute name="VALUE" x="-1680.436" y="-856.282" size="1.778" layer="96" rot="R180"/>
+</instance>
+<instance part="GND1" gate="1" x="-1679.5" y="-906.3" smashed="yes">
+<attribute name="VALUE" x="-1682.04" y="-908.84" size="1.778" layer="96"/>
+</instance>
+<instance part="GND2" gate="1" x="-1818.7" y="-908" smashed="yes">
+<attribute name="VALUE" x="-1821.24" y="-910.54" size="1.778" layer="96"/>
+</instance>
 </instances>
 <busses>
@@
 <pinref part="CHIP" gate="G$1" pin="1"/>
 <pinref part="C1" gate="C1" pin="2"/>
-<wire x1="-1779.88" y1="-863.17" x2="-1805.6" y2="-863.37" width="0.1524" layer="91"/>
-<wire x1="-1805.6" y1="-863.37" x2="-1805.6" y2="-878.22" width="0.1524" layer="91"/>
+<wire x1="-1779.88" y1="-863.17" x2="-1805.6" y2="-863.17" width="0.1524" layer="91"/>
+<wire x1="-1805.6" y1="-863.17" x2="-1805.6" y2="-863.26" width="0.1524" layer="91"/>
+<pinref part="J1" gate="G$1" pin="1"/>
+<wire x1="-1805.6" y1="-863.3" x2="-1805.6" y2="-878.22" width="0.1524" layer="91"/>
+<wire x1="-1815.56" y1="-863.26" x2="-1805.6" y2="-863.26" width="0.1524" layer="91"/>
+<wire x1="-1805.6" y1="-863.26" x2="-1805.6" y2="-863.3" width="0.1524" layer="91"/>
+<junction x="-1805.6" y="-863.3"/>
 </segment>
 </net>
@@
 <pinref part="CHIP" gate="G$1" pin="2"/>
 <pinref part="C2" gate="C1" pin="2"/>
-<wire x1="-1744.22" y1="-863.26" x2="-1728.4" y2="-863.46" width="0.1524" layer="91"/>
-<wire x1="-1728.4" y1="-863.46" x2="-1728.4" y2="-863.5" width="0.1524" layer="91"/>
+<wire x1="-1744.22" y1="-863.26" x2="-1728.4" y2="-863.26" width="0.1524" layer="91"/>
+<wire x1="-1728.4" y1="-863.26" x2="-1728.4" y2="-863.1" width="0.1524" layer="91"/>
 <pinref part="C3" gate="C1" pin="2"/>
-<wire x1="-1728.4" y1="-863.5" x2="-1728.4" y2="-876.22" width="0.1524" layer="91"/>
-<wire x1="-1700.2" y1="-867.02" x2="-1700.2" y2="-863.5" width="0.1524" layer="91"/>
-<wire x1="-1700.2" y1="-863.5" x2="-1728.4" y2="-863.5" width="0.1524" layer="91"/>
-<junction x="-1728.4" y="-863.5"/>
+<wire x1="-1728.4" y1="-863.1" x2="-1728.4" y2="-876.22" width="0.1524" layer="91"/>
+<wire x1="-1700.2" y1="-867.02" x2="-1700.2" y2="-863.1" width="0.1524" layer="91"/>
+<wire x1="-1700.2" y1="-863.1" x2="-1728.4" y2="-863.1" width="0.1524" layer="91"/>
+<junction x="-1728.4" y="-863.1"/>
+<pinref part="J2" gate="G$1" pin="1"/>
+<wire x1="-1687.04" y1="-863.14" x2="-1700.3" y2="-863.14" width="0.1524" layer="91"/>
+<wire x1="-1700.3" y1="-863.14" x2="-1700.2" y2="-863.1" width="0.1524" layer="91"/>
+<junction x="-1700.2" y="-863.1"/>
 </segment>
 </net>
@@
 </segment>
 </net>
-<net name="N$6" class="0">
+<net name="GND" class="0">
+<segment>
+<pinref part="CHIP" gate="G$1" pin="4"/>
+<wire x1="-1779.78" y1="-870.88" x2="-1779.78" y2="-903.9" width="0.1524" layer="91"/>
+<wire x1="-1779.78" y1="-903.9" x2="-1805.6" y2="-903.9" width="0.1524" layer="91"/>
+<pinref part="C1" gate="C1" pin="1"/>
+<wire x1="-1805.6" y1="-903.9" x2="-1805.6" y2="-890.92" width="0.1524" layer="91"/>
+<pinref part="GND2" gate="1" pin="GND"/>
+<wire x1="-1818.7" y1="-905.46" x2="-1818.7" y2="-903.9" width="0.1524" layer="91"/>
+<wire x1="-1818.7" y1="-903.9" x2="-1805.6" y2="-903.9" width="0.1524" layer="91"/>
+<junction x="-1805.6" y="-903.9"/>
+</segment>
 <segment>
 <pinref part="CHIP" gate="G$1" pin="3"/>
-<wire x1="-1744.22" y1="-870.88" x2="-1744.72" y2="-903.8" width="0.1524" layer="91"/>
-<wire x1="-1744.72" y1="-903.8" x2="-1728.4" y2="-903.8" width="0.1524" layer="91"/>
+<wire x1="-1744.22" y1="-870.88" x2="-1744.12" y2="-903" width="0.1524" layer="91"/>
+<wire x1="-1744.12" y1="-903" x2="-1728.4" y2="-903.1" width="0.1524" layer="91"/>
 <pinref part="C4" gate="C1" pin="1"/>
-<wire x1="-1728.4" y1="-903.8" x2="-1700.2" y2="-903.8" width="0.1524" layer="91"/>
-<wire x1="-1700.2" y1="-903.8" x2="-1700.2" y2="-897.22" width="0.1524" layer="91"/>
+<wire x1="-1728.4" y1="-903.1" x2="-1700.2" y2="-903" width="0.1524" layer="91"/>
+<wire x1="-1700.2" y1="-903" x2="-1700.2" y2="-897.22" width="0.1524" layer="91"/>
 <pinref part="C2" gate="C1" pin="1"/>
-<wire x1="-1728.4" y1="-888.92" x2="-1728.4" y2="-903.8" width="0.1524" layer="91"/>
-</segment>
-</net>
-<net name="N$7" class="0">
-<segment>
-<pinref part="CHIP" gate="G$1" pin="4"/>
-<wire x1="-1779.78" y1="-870.88" x2="-1780.48" y2="-903.8" width="0.1524" layer="91"/>
-<wire x1="-1780.48" y1="-903.8" x2="-1805.8" y2="-903.8" width="0.1524" layer="91"/>
-<pinref part="C1" gate="C1" pin="1"/>
-<wire x1="-1805.8" y1="-903.8" x2="-1805.6" y2="-890.92" width="0.1524" layer="91"/>
+<wire x1="-1728.4" y1="-888.92" x2="-1728.4" y2="-903.1" width="0.1524" layer="91"/>
+<pinref part="GND1" gate="1" pin="GND"/>
+<wire x1="-1679.5" y1="-903.76" x2="-1679.5" y2="-903" width="0.1524" layer="91"/>
+<wire x1="-1679.5" y1="-903" x2="-1700.2" y2="-903" width="0.1524" layer="91"/>
+<junction x="-1700.2" y="-903"/>
 </segment>
 </net>
@@
 </schematic>
 </drawing>
+<compatibility>
+<note version="8.2" severity="warning">
+Since Version 8.2, EAGLE supports online libraries. The ids
+of those online libraries will not be understood (or retained)
+with this version.
+</note>
+<note version="8.3" severity="warning">
+Since Version 8.3, EAGLE supports URNs for individual library
+assets (packages, symbols, and devices). The URNs of those assets
+will not be understood (or retained) with this version.
+</note>
+</compatibility>
 </eagle>
