File: Thesis Work/Layout/PCB Design/Eagle/DM & CM/DMP2.brd (EAGLE design)
At the start: 72.5 x 36 mm, 12 parts, among them J1 SMA-J-P-H-ST-EM1, J2 SMA-J-P-H-ST-EM1, J3 SMA-J-P-H-ST-EM1, J4 SMA-J-P-H-ST-EM1

Commit message: c
Parts:
- moved J4 6.95 mm to (75.0, 13.1)
- moved JP1 5.44 mm to (61.0, 16.0)
- moved J3 5.40 mm to (75.0, 32.6)
- moved J1 5.00 mm to (20.0, 33.0)
- moved J2 5.00 mm to (20.0, 12.5)
- moved C5 2.98 mm to (64.0, 29.1)
- moved C4 1.80 mm to (53.6, 20.5)
- moved C3 1.70 mm to (53.5, 25.3)
- moved C1 1.30 mm to (28.9, 22.9)
Routing:
- net N$7: track 214.5 -> 0.00 mm
- net N$5: track 18.3 -> 23.2 mm
- net N$3: track 17.9 -> 22.4 mm
- net N$1: track 44.6 -> 40.9 mm
- net N$2: track 3.26 -> 6.26 mm
- net N$6: track 2.86 -> 3.59 mm
- net N$4: track 41.8 -> 42.4 mm
- added copper zone on layer 16, net GND
Other:
- board size 72.5 x 36 mm -> 65.6 x 39 mm
